File: 100100mm/Statikplatte.sch (KiCad schematic (older format))
At the start: 31 parts, among them J1 VIN, J10 HV, J2 GND, J3 GND, J4 GND, J5 GND, J6 GND, J7 HV, J8 HV, J9 HV

Commit message: updated boards
Parts:
- D1, D10, D2, D3, D4, D5, D6, D7, D8, D9: value D -> SS34
Changed lines of the file:
@@
 EESchema Schematic File Version 4
+LIBS:Statikplatte-cache
 EELAYER 26 0
 EELAYER END
@@
 P 4450 3600
 F 0 "D1" V 4404 3679 50  0000 L CNN
-F 1 "D" V 4495 3679 50  0000 L CNN
+F 1 "SS34" V 4495 3679 50  0000 L CNN
 F 2 "otter:SMAF" H 4450 3600 50  0001 C CNN
 F 3 "~" H 4450 3600 50  0001 C CNN
@@
 P 4950 3600
 F 0 "D2" V 4996 3521 50  0000 R CNN
-F 1 "D" V 4905 3521 50  0000 R CNN
+F 1 "SS34" V 4905 3521 50  0000 R CNN
 F 2 "otter:SMAF" H 4950 3600 50  0001 C CNN
 F 3 "~" H 4950 3600 50  0001 C CNN
@@
 P 5500 3600
 F 0 "D3" V 5454 3679 50  0000 L CNN
-F 1 "D" V 5545 3679 50  0000 L CNN
+F 1 "SS34" V 5545 3679 50  0000 L CNN
 F 2 "otter:SMAF" H 5500 3600 50  0001 C CNN
 F 3 "~" H 5500 3600 50  0001 C CNN
@@
 P 6000 3600
 F 0 "D4" V 6046 3521 50  0000 R CNN
-F 1 "D" V 5955 3521 50  0000 R CNN
+F 1 "SS34" V 5955 3521 50  0000 R CNN
 F 2 "otter:SMAF" H 6000 3600 50  0001 C CNN
 F 3 "~" H 6000 3600 50  0001 C CNN
@@
 P 6550 3600
 F 0 "D5" V 6504 3679 50  0000 L CNN
-F 1 "D" V 6595 3679 50  0000 L CNN
+F 1 "SS34" V 6595 3679 50  0000 L CNN
 F 2 "otter:SMAF" H 6550 3600 50  0001 C CNN
 F 3 "~" H 6550 3600 50  0001 C CNN
@@
 P 7050 3600
 F 0 "D6" V 7096 3521 50  0000 R CNN
-F 1 "D" V 7005 3521 50  0000 R CNN
+F 1 "SS34" V 7005 3521 50  0000 R CNN
 F 2 "otter:SMAF" H 7050 3600 50  0001 C CNN
 F 3 "~" H 7050 3600 50  0001 C CNN
@@
 P 7600 3600
 F 0 "D7" V 7554 3679 50  0000 L CNN
-F 1 "D" V 7645 3679 50  0000 L CNN
+F 1 "SS34" V 7645 3679 50  0000 L CNN
 F 2 "otter:SMAF" H 7600 3600 50  0001 C CNN
 F 3 "~" H 7600 3600 50  0001 C CNN
@@
 P 8100 3600
 F 0 "D8" V 8146 3521 50  0000 R CNN
-F 1 "D" V 8055 3521 50  0000 R CNN
+F 1 "SS34" V 8055 3521 50  0000 R CNN
 F 2 "otter:SMAF" H 8100 3600 50  0001 C CNN
 F 3 "~" H 8100 3600 50  0001 C CNN
@@
 P 8650 3600
 F 0 "D9" V 8604 3679 50  0000 L CNN
-F 1 "D" V 8695 3679 50  0000 L CNN
+F 1 "SS34" V 8695 3679 50  0000 L CNN
 F 2 "otter:SMAF" H 8650 3600 50  0001 C CNN
 F 3 "~" H 8650 3600 50  0001 C CNN
@@
 P 9150 3600
 F 0 "D10" V 9196 3521 50  0000 R CNN
-F 1 "D" V 9105 3521 50  0000 R CNN
+F 1 "SS34" V 9105 3521 50  0000 R CNN
 F 2 "otter:SMAF" H 9150 3600 50  0001 C CNN
 F 3 "~" H 9150 3600 50  0001 C CNN
