File: 5050mm/Statikplatte.kicad_pcb (KiCad board)
At the start: 4 copper layers, 50 x 50 mm, 24 parts, among them J10 HV, J11 SCREW, J2 GND, J3 IN+, J4 GND, J5 GND, J6 GND, J7 HV, J8 HV, J9 HV

Commit message: updated boards
Parts:
- removed J11: SCREW, otter:M3_Screw
Routing:
- net /GNDE: track 70.7 -> 3.32 mm, vias 3 -> 5
- net /HV: track 53.4 -> 94.8 mm, vias 2 -> 1
Other:
- board text added: "50*50mm | 1.5*0.5mm"
- board text added: "Design by Jana Marie Hemsing"
- board text removed: "50*50mm | 0.5*0.5mm"
- board text removed: "Design by Jan Henrik Hemsing"

Commit message: added images
Other:
- board text removed: "1 F.Cu"
- board text removed: "2 In1.Cu"
- board text removed: "3 In2.Cu"
- board text removed: "4 B.Cu"
Changed lines of the file:
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@@
   (general
     (thickness 1.6)
-    (drawings 21)
+    (drawings 17)
     (tracks 78)
     (zones 0)
@@
       (net 6 /N1))
   )
-  (gr_text "4 B.Cu" (at 119 83) (layer B.Cu)
-    (effects (font (size 1.5 1.5) (thickness 0.35)))
-  )
-  (gr_text "3 In2.Cu" (at 119 81) (layer In2.Cu)
-    (effects (font (size 1.5 1.5) (thickness 0.3)))
-  )
-  (gr_text "2 In1.Cu\n" (at 119 79) (layer In1.Cu)
-    (effects (font (size 1.5 1.5) (thickness 0.3)))
-  )
-  (gr_text "1 F.Cu\n" (at 119 77) (layer F.Cu)
-    (effects (font (size 1.5 1.5) (thickness 0.3)))
-  )
   (gr_text "50*50mm | 1.5*0.5mm" (at 150 86.8) (layer B.SilkS)

Commit message: updated to KICAD 6
Other:
- net class Default removed
