File: DINA5/Statikplatte.kicad_pcb (KiCad board)
At the start: 2 copper layers, 210 x 148 mm, 35 parts, among them J10 HV, J11 SCREW, J12 SCREW, J13 SCREW, J14 SCREW, J2 GND, J3 IN+, J4 GND, J5 GND, J6 GND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

Commit message: updated design
Parts:
- moved J10 6.00 mm to (15.0, 104.0), turned to 0 degrees
- moved J2 6.00 mm to (105.0, 163.0), turned to 90 degrees
- moved J4 6.00 mm to (225.0, 74.0)
- moved J5 6.00 mm to (105.0, 15.0)
- moved J6 6.00 mm to (15.0, 74.0), turned to 0 degrees
- moved J7 6.00 mm to (135.0, 163.0), turned to 90 degrees
- moved J8 6.00 mm to (135.0, 15.0), turned to 270 degrees
- moved J9 6.00 mm to (225.0, 104.0)
Routing:
- net /GNDE: track 355.7 -> 361.7 mm
- net /HV: track 330.6 -> 333.7 mm
Other:
- board text added: "Design by Jana Marie Hemsing 2021"
- board text removed: "Design by Jan Henrik Hemsing and Niklas Fauth"

Commit message: updated to KICAD 6
Other:
- net class Default removed
